File: hw/sch_pcb/TFHT01A.kicad_pcb (KiCad board)
At the start: 2 copper layers, 37.5 x 19 mm, 23 parts, among them J1 HEADER_1x03, J2 SM04B-GHS-TB, J3 SM04B-GHS-TB, M2 M3, U1 PCF8583, U2 74HC1G14GW, U3 MIC5504-3.3YM5

Commit message: Edit PCB
Parts:
- removed C2: 10uF, Mlab_R:SMD-0805
- removed C6: 100nF, Mlab_R:SMD-0603
- removed G***: LOGO, MLAB_LOGA:TF
- removed J3: SM04B-GHS-TB, Connector_JST:JST_GH_SM04B-GHS-TB_1x04-1MP_P1.25mm_Horizontal
- removed JP2: SolderJumper_3_Bridged12, Jumper:SolderJumper-3_P1.3mm_Bridged12_RoundedPad1.0x1.5mm
- removed U2: 74HC1G14GW, Package_TO_SOT_SMD:SOT-353_SC-70-5
- added D3: LED RED, Mlab_D:LED_1206, B.Cu at (8.50, -2.00)
- added M1: M3, Mlab_Mechanical:dira_3mm, F.Cu at (22.5, -15.0)
- added M3: M3, Mlab_Mechanical:dira_3mm, F.Cu at (2.50, 0.00)
- added M4: M3, Mlab_Mechanical:dira_3mm, F.Cu at (12.5, -15.0)
- added M5: M3, Mlab_Mechanical:dira_3mm, F.Cu at (22.5, 0.00)
- added M6: M3, Mlab_Mechanical:dira_3mm, F.Cu at (2.50, -15.0)
- added Q1: BC817, Package_TO_SOT_SMD:SOT-23, B.Cu at (16.9, -3.05)
- D1: value ZENER-5.6V -> BZX585-B5V6.115; footprint Mlab_D:Diode-MiniMELF_Standard -> Diode_SMD:D_SOD-523
- D2: value LED RED -> LED GREEN
- J1: value HEADER_1x03 -> SM04B-GHS-TB; footprint Connector_PinHeader_2.54mm:PinHeader_1x03_P2.54mm_Horizontal -> Connector_JST:JST_GH_SM04B-GHS-TB_1x04-1MP_P1.25mm_Horizontal
- J2: moved to F.Cu
- M2: footprint Mlab_Mechanical:MountingHole_3mm -> Mlab_Mechanical:dira_3mm; moved to F.Cu
- R1: value 470R -> 180R; footprint Mlab_R:SMD-0805 -> Mlab_R:SMD-0603
- R2: footprint Mlab_R:SMD-0805 -> Mlab_R:SMD-0603
- U1: value PCF8583 -> SHT31; footprint Mlab_IO:SOT176-1 -> Mlab_IO:DFN-8-1EP_2.4x2.4mm_Pitch0.5mm
- moved D2 196.9 mm to (8.50, -13.0), turned to 180 degrees
- moved J1 196.5 mm to (2.80, -7.50), turned to 90 degrees
- moved R2 185.2 mm to (14.4, -11.9), turned to 0 degrees
- moved JP1 182.8 mm to (19.6, -8.89)
- moved D1 180.6 mm to (7.37, -10.1), turned to 90 degrees
- moved C1 180.1 mm to (11.3, -9.50)
- moved R4 179.2 mm to (20.3, -2.79), turned to 0 degrees
- moved C5 179.0 mm to (18.3, -12.1)
- moved R1 178.9 mm to (21.6, -6.10), turned to 0 degrees
- moved M2 178.7 mm to (12.5, 0.00)
- moved U3 177.0 mm to (8.51, -6.10), turned to 90 degrees
- moved C3 175.0 mm to (9.53, -9.84)
- moved J2 174.4 mm to (2.80, -7.50), turned to -90 degrees
- moved R3 173.0 mm to (19.4, -12.2), turned to 0 degrees
- moved U1 172.5 mm to (27.0, -7.50), turned to 90 degrees
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Connections:
- J1 pad 1: /COUNT -> +5V
- J1 pad 2: Net-(C2-Pad1) -> /SCL
- J1 pad 3: GND -> /SDA
- R1 pad 1: Net-(JP2-Pad2) -> +5V
- R1 pad 2: /COUNT -> Net-(D2-Pad2)
- R10 pad 2: /SCL -> /SDA
- R2 pad 1: Net-(C2-Pad1) -> /ALERT
- R2 pad 2: Net-(JP2-Pad2) -> Net-(Q1-Pad1)
- R3 pad 2: /SDA -> /SCL
- R4 pad 1: Net-(R4-Pad1) -> Net-(D3-Pad1)
- R4 pad 2: Net-(D2-Pad2) -> Net-(Q1-Pad3)
- U1 pad 1: Net-(R4-Pad1) -> /SDA
- U1 pad 2: (no net) -> Net-(JP1-Pad2)
- U1 pad 3: Net-(JP1-Pad2) -> /ALERT
- U1 pad 4: GND -> /SCL
- U1 pad 5: /SDA -> +3V3
- U1 pad 6: /SCL -> unconnected-(U1-Pad6)
- U1 pad 7: (no net) -> GND
- U1 pad 8: +3V3 -> GND
- U3 pad 4: (no net) -> unconnected-(U3-Pad4)
Routing:
- net +5V: track 45.8 -> 0.00 mm, vias 4 -> 0
- net +3V3: track 38.4 -> 0.00 mm, vias 3 -> 0
- net /SCL: track 27.9 -> 0.00 mm
- net /SDA: track 25.6 -> 0.00 mm, vias 2 -> 0
- net Net-(R4-Pad1): track 18.9 -> 0.00 mm
- net Net-(JP1-Pad2): track 13.9 -> 0.00 mm
- net /COUNT: track 12.6 -> 0.00 mm
- net Net-(JP2-Pad2): track 10.5 -> 0.00 mm
- net Net-(C2-Pad1): track 9.86 -> 0.00 mm
- net Net-(D2-Pad2): track 2.16 -> 0.00 mm
- net GND: vias 60 -> 0
- removed copper zone on B.Cu, net GND
- removed copper zone on F.Cu, net GND
Other:
- board size 37.5 x 19 mm -> 30 x 15 mm
- board text removed: "+5V"
- board text removed: "0X50"
- board text removed: "2021"
- board text removed: "GND"
- board text removed: "I2C"
- board text removed: "IN"
- board text removed: "PULSE"
- board text removed: "TFRPM01C"
- board text removed: "ThunderFly.cz"

Commit message: Edit PCB
Parts:
- added G***: LOGO, MLAB_LOGA:TF, F.Cu at (17.0, -9.14)
- moved R1 9.29 mm to (13.3, -10.3), turned to 90 degrees
- moved C5 8.67 mm to (26.9, -11.0)
- moved R2 7.66 mm to (18.4, -5.33), turned to 180 degrees
- moved JP1 7.03 mm to (18.0, -2.03), turned to 180 degrees
- moved R4 6.99 mm to (13.3, -2.67)
- moved R10 4.67 mm to (15.5, -10.3), turned to -90 degrees
- moved Q1 3.35 mm to (14.9, -5.71), turned to 180 degrees
- moved R3 2.52 mm to (17.8, -10.3), turned to -90 degrees
- moved C4 0.63 mm to (11.8, -5.36)
- moved U3 0.51 mm to (9.02, -6.10)
Routing:
- net /SDA: track 0.00 -> 33.3 mm, vias 0 -> 4
- net +5V: track 0.00 -> 29.9 mm, vias 0 -> 2
- net /SCL: track 0.00 -> 29.4 mm, vias 0 -> 2
- net +3V3: track 0.00 -> 29.2 mm
- net GND: track 0.00 -> 24.3 mm, vias 0 -> 33
- net Net-(JP1-Pad2): track 0.00 -> 14.1 mm
- net /ALERT: track 0.00 -> 10.6 mm
- net Net-(D3-Pad1): track 0.00 -> 8.74 mm, vias 0 -> 2
- net Net-(D2-Pad2): track 0.00 -> 3.55 mm
- net Net-(Q1-Pad3): track 0.00 -> 3.15 mm
- net Net-(Q1-Pad1): track 0.00 -> 2.32 mm
- added copper zone on B.Cu, net GND
- added copper zone on F.Cu, net GND
Other:
- board text added: "TFHT01A"
